Commit message: fix: 修复IK求解x0 is infeasible错误 - 裁剪种子点+奇异点处理

File: config/piper_description.urdf (robot description, URDF)
Before this commit: robot piper, 11 links, 10 joints
Links:
- removed link dummy_link
- link base_link: geometry collision mesh filename=package://piper_description/meshes/base_link.STL; visual mesh filename=package://piper_description/meshes/base_link.STL
- link gripper_base: geometry collision mesh filename=package://piper_description/meshes/gripper_base.STL; visual mesh filename=package://piper_description/meshes/gripper_base.STL
- link link1: geometry collision mesh filename=package://piper_description/meshes/link1.STL; visual mesh filename=package://piper_description/meshes/link1.STL
- link link2: geometry collision mesh filename=package://piper_description/meshes/link2.STL; visual mesh filename=package://piper_description/meshes/link2.STL
- link link3: geometry collision mesh filename=package://piper_description/meshes/link3.STL; visual mesh filename=package://piper_description/meshes/link3.STL
- link link4: geometry collision mesh filename=package://piper_description/meshes/link4.STL; visual mesh filename=package://piper_description/meshes/link4.STL
- link link5: geometry collision mesh filename=package://piper_description/meshes/link5.STL; visual mesh filename=package://piper_description/meshes/link5.STL
- link link6: mass 0.007 -> 0.00699089613564366; geometry collision mesh filename=package://piper_description/meshes/link6.STL; visual mesh filename=package://piper_description/meshes/link6.STL
- link link7: geometry collision mesh filename=package://piper_description/meshes/link7.STL; visual mesh filename=package://piper_description/meshes/link7.STL
- link link8: geometry collision mesh filename=package://piper_description/meshes/link8.STL; visual mesh filename=package://piper_description/meshes/link8.STL
Joints:
- removed joint base_to_dummy
